File: _autosave-LNWB_BJT.kicad_pcb (KiCad board)
At the start: 4 copper layers, 75 x 50 mm, 116 parts, among them J1 Input, J2 wire2board, J3 Input, J4 wire2board, Q1 2N4401, Q2 2N4401, Q3 2N3906, Q4 BD679, Q5 BD680, U1 TL072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

Commit message: send.
Parts:
- moved C21 1.50 mm to (100.1, 86.5)
- moved C19 0.50 mm to (96.7, 88.4)
Routing:
- net Net-(PS1-+Vout): track 0.00 -> 11.6 mm
- net +5V: track 9.43 -> 17.5 mm
- net GND: track 45.5 -> 48.4 mm, vias 36 -> 39
- net Net-(C4-Pad1): track 0.00 -> 1.78 mm
Changed lines of the file:
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@@
 	(footprint "Capacitor_THT:CP_Radial_D5.0mm_P2.00mm"
 		(layer "F.Cu")
-		(at 96.955112 88 180)
+		(at 96.655113 88.4 180)
 		(descr "CP, Radial series, Radial, pin pitch=2.00mm, , diameter=5mm, Electrolytic Capacitor")
 		(tags "CP Radial series Radial pin pitch 2.00mm  diameter 5mm Electrolytic Capacitor")
@@
 	(footprint "Resistor_SMD:R_0603_1608Metric_Pad0.98x0.95mm_HandSolder"
 		(layer "F.Cu")
-		(at 100 85 180)
+		(at 100.1 86.5 180)
 		(descr "Resistor SMD 0603 (1608 Metric), square (rectangular) end terminal, IPC_7351 nominal with elongated pad for handsoldering. (Body size source: IPC-SM-782 page 72, https://www.pcb-3d.com/wordpress/wp-content/uploads/ipc-sm-782a_amendment_1_and_2.pdf), generated with kicad-footprint-generator")
 		(tags "resistor handsolder")
@@
 	)
 	(segment
+		(start 87.3625 94)
+		(end 89.1375 94)
+		(width 0.5)
+		(layer "F.Cu")
+		(net 5)
+	)
+	(segment
 		(start 83.9125 92)
 		(end 83.9125 94)
@@
 	)
 	(segment
+		(start 104.4575 81.505)
+		(end 104.55 81.4125)
+		(width 0.5)
+		(layer "F.Cu")
+		(net 12)
+	)
+	(segment
+		(start 100.55 81.505)
+		(end 104.4575 81.505)
+		(width 0.5)
+		(layer "F.Cu")
+		(net 12)
+	)
+	(segment
+		(start 104.55 85.275)
+		(end 107.17 87.895)
+		(width 0.5)
+		(layer "F.Cu")
+		(net 12)
+	)
+	(segment
+		(start 104.55 81.4125)
+		(end 104.55 85.275)
+		(width 0.5)
+		(layer "F.Cu")
+		(net 12)
+	)
+	(segment
 		(start 110 92.9125)
 		(end 110 94.5875)
@@
 	)
 	(segment
+		(start 99.1125 88.4)
+		(end 96.655113 88.4)
+		(width 0.5)
+		(layer "F.Cu")
+		(net 15)
+	)
+	(segment
+		(start 101.0125 86.5)
+		(end 99.1125 88.4)
+		(width 0.5)
+		(layer "F.Cu")
+		(net 15)
+	)
+	(segment
+		(start 101.0125 86.5)
+		(end 101.0125 84.2475)
+		(width 0.5)
+		(layer "F.Cu")
+		(net 15)
+	)
+	(segment
 		(start 82.4875 78.7)
 		(end 80.595 80.5925)
@@
 		(net 15)
 	)
+	(segment
+		(start 101.0125 84.2475)
+		(end 100.55 83.785)
+		(width 0.5)
+		(layer "F.Cu")
+		(net 15)
+	)
 	(via
 		(at 78 83)
@@
 	)
 	(segment
+		(start 104.5 100.7)
+		(end 104.5 101.6875)
+		(width 0.5)
+		(layer "F.Cu")
+		(net 28)
+	)
+	(segment
 		(start 96 108.5675)
 		(end 96.52 109.0875)
@@
 	)
 	(segment
+		(start 103 100.7)
+		(end 103 101.6875)
+		(width 0.5)
+		(layer "F.Cu")
+		(net 28)
+	)
+	(segment
 		(start 107.4125 115)
 		(end 108.4 115)
@@
 	)
 	(segment
+		(start 106 100.7)
+		(end 106 101.6875)
+		(width 0.5)
+		(layer "F.Cu")
+		(net 28)
+	)
+	(segment
 		(start 110.0875 100)
 		(end 110 99.9125)
@@
 	)
 	(via
+		(at 106 100.7)
+		(size 0.6)
+		(drill 0.3)
+		(layers "F.Cu" "B.Cu")
+		(net 28)
+	)
+	(via
 		(at 97 123.4)
 		(size 0.6)
@@
 		(size 0.6)
 		(drill 0.3)
+		(layers "F.Cu" "B.Cu")
+		(net 28)
+	)
+	(via
+		(at 104.5 100.7)
+		(size 0.6)
+		(drill 0.3)
+		(layers "F.Cu" "B.Cu")
+		(net 28)
+	)
+	(via
+		(at 103 100.7)
+		(size 0.6)
+		(drill 0.3)
