File: LNWB_BJT.kicad_pcb (KiCad board)
At the start: 4 copper layers, 75 x 50 mm, 116 parts, among them J1 Input, J2 wire2board, J3 Input, J4 wire2board, Q1 2N4401, Q2 2N4401, Q3 2N3906, Q4 BD679, Q5 BD680, U1 TL072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

Commit message: PCB.
Parts:
- D3, D4: moved to B.Cu
- moved J4 6.50 mm to (123.5, 91.5)
- moved D3 2.50 mm to (78.5, 114.7)
- moved D4 2.50 mm to (76.0, 122.3)
- moved C16 2.12 mm to (105.5, 82.4), turned to 0 degrees
- moved Q4 1.70 mm to (100.5, 77.5)
- moved C21 1.50 mm to (100.1, 86.5)
- moved R17 1.50 mm to (103.0, 77.0)
- moved C17 1.29 mm to (107.4, 79.3), turned to 90 degrees
- moved FB9 1.06 mm to (113.8, 82.2)
- moved C19 0.85 mm to (96.7, 87.2)
- moved R25 0.60 mm to (110.5, 110.6)
- moved R24 0.50 mm to (110.5, 109.0)
- moved C24 0.40 mm to (96.9, 110.0)
- moved C27 0.40 mm to (93.9, 110.0)
- moved FB1 0.40 mm to (99.4, 111.0)
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Connections:
- FB9 pad 1: 0 -> GND
Routing:
- net +5V: track 9.43 -> 65.2 mm, vias 2 -> 5
- net Earth: track 0.00 -> 28.3 mm, vias 0 -> 1
- net Net-(J2-Pin_1): track 0.00 -> 18.4 mm
- net Net-(PS1-+Vout): track 0.00 -> 13.4 mm
- net GND: track 45.5 -> 55.2 mm, vias 36 -> 44
- net Net-(Q4-B): track 0.00 -> 8.84 mm
- net -5V: track 10.2 -> 18.9 mm, vias 1 -> 4
- net Net-(C2-Pad2): track 0.00 -> 5.31 mm
- net Net-(J1-In): track 0.00 -> 5.19 mm
- net Net-(U2A-+): track 42.5 -> 46.6 mm, vias 2 -> 1
- net Net-(Q2-C): track 18.4 -> 20.2 mm, vias 1 -> 2
- net Net-(C4-Pad1): track 0.00 -> 1.78 mm
- net Net-(U1A--): track 31.3 -> 29.8 mm
- added copper zone on In2.Cu, net +5V
- added copper zone on B.Cu, net -5V
